File: pokecom_cas_if.kicad_pcb (KiCad board)
At the start: 2 copper layers, 40 x 50 mm, 17 parts, among them J1 Conn_01x11, J2 Conn_01x11, J3 Conn_01x05, J4 SJ1-3525N, J5 USB_B_Micro

Commit message: update Ver2.0
Parts:
- added R5: 56k, Resistor_THT:R_Axial_DIN0207_L6.3mm_D2.5mm_P7.62mm_Horizontal, F.Cu at (-334.5, -533.0)
- added R6: 56k, Resistor_THT:R_Axial_DIN0207_L6.3mm_D2.5mm_P7.62mm_Horizontal, F.Cu at (-334.5, -525.0)
- added R7: 560, Resistor_THT:R_Axial_DIN0207_L6.3mm_D2.5mm_P7.62mm_Horizontal, F.Cu at (-350.5, -535.5)
- added R8: 560, Resistor_THT:R_Axial_DIN0207_L6.3mm_D2.5mm_P7.62mm_Horizontal, F.Cu at (-350.6, -541.0)
- C1, C2, C3, C4: footprint C_Rect_L7.0mm_W3.5mm_P5.00mm -> Capacitor_THT:C_Rect_L7.0mm_W3.5mm_P5.00mm
- moved R3 2.50 mm to (-347.0, -533.0)
- moved R4 2.50 mm to (-347.0, -538.5)
Routing:
- net /+5V: track 28.4 -> 79.9 mm
- net /VGG: track 48.6 -> 79.6 mm
- net Net-(C2-Pad1): track 41.4 -> 36.3 mm
- net Net-(C3-Pad1): track 19.4 -> 23.5 mm
- net Net-(C2-Pad2): track 3.62 -> 7.62 mm
- net /Xout: track 17.8 -> 21.6 mm
- net Net-(C1-Pad2): track 30.0 -> 33.5 mm
- net /Xin: track 12.6 -> 14.2 mm
