File: pokecom_cas_if.sch (KiCad schematic (older format))
At the start: 13 parts, among them J1 Conn_01x11, J2 Conn_01x11, J3 Conn_01x05, J4 SJ1-3525N, J5 USB_B_Micro

Commit message: update Ver2.0
Parts:
- added R5, R6: 56k, Resistor_THT:R_Axial_DIN0207_L6.3mm_D2.5mm_P7.62mm_Horizontal, symbol Device:R
- added R7, R8: 560, Resistor_THT:R_Axial_DIN0207_L6.3mm_D2.5mm_P7.62mm_Horizontal, symbol Device:R
- C1, C2, C3, C4: footprint :C_Rect_L7.0mm_W3.5mm_P5.00mm -> Capacitor_THT:C_Rect_L7.0mm_W3.5mm_P5.00mm
Connections:
- net +5V: now also R7.1, R8.1
- net Xin: now also R5.2
- net Xout: now also R6.2
- net at C2.1, C4.1, J4.2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: now also R8.2
- net at C3.1, J4.3, R3.1: now also R7.2
- net at C2.2, R1.1: now also R5.1
- net at C1.2, C3.2, R2.1: now also R6.1
Changed lines of the file:
@@
 F 0 "C2" V 4748 4000 50  0000 C CNN
 F 1 "0.047u" V 4839 4000 50  0000 C CNN
-F 2 ":C_Rect_L7.0mm_W3.5mm_P5.00mm" H 5038 3850 50  0001 C CNN
+F 2 "Capacitor_THT:C_Rect_L7.0mm_W3.5mm_P5.00mm" H 5038 3850 50  0001 C CNN
 F 3 "~" H 5000 4000 50  0001 C CNN
 	1    5000 4000
@@
 F 0 "C3" V 4748 4450 50  0000 C CNN
 F 1 "0.047u" V 4839 4450 50  0000 C CNN
-F 2 ":C_Rect_L7.0mm_W3.5mm_P5.00mm" H 5038 4300 50  0001 C CNN
+F 2 "Capacitor_THT:C_Rect_L7.0mm_W3.5mm_P5.00mm" H 5038 4300 50  0001 C CNN
 F 3 "~" H 5000 4450 50  0001 C CNN
 	1    5000 4450
@@
 F 0 "C4" H 5185 3604 50  0000 R CNN
 F 1 "0.047u" H 5185 3695 50  0000 R CNN
-F 2 ":C_Rect_L7.0mm_W3.5mm_P5.00mm" H 5338 3500 50  0001 C CNN
+F 2 "Capacitor_THT:C_Rect_L7.0mm_W3.5mm_P5.00mm" H 5338 3500 50  0001 C CNN
 F 3 "~" H 5300 3650 50  0001 C CNN
 	1    5300 3650
@@
 F 0 "C1" H 4665 3696 50  0000 L CNN
 F 1 "0.047u" H 4665 3605 50  0000 L CNN
-F 2 ":C_Rect_L7.0mm_W3.5mm_P5.00mm" H 4588 3500 50  0001 C CNN
+F 2 "Capacitor_THT:C_Rect_L7.0mm_W3.5mm_P5.00mm" H 4588 3500 50  0001 C CNN
 F 3 "~" H 4550 3650 50  0001 C CNN
 	1    4550 3650
@@
 	2750 3100 3600 3100
 Wire Wire Line
-	3600 3100 3600 4000
+	3600 3100 3600 3650
 Wire Wire Line
 	5150 4000 5300 4000
@@
 	6400 4300 6550 4300
 Wire Wire Line
-	5150 4450 5750 4450
+	5150 4450 5550 4450
 Wire Wire Line
 	4850 4450 4550 4450
@@
 Connection ~ 5300 4000
 Wire Wire Line
-	5300 4000 6100 4000
+	5300 4000 5950 4000
 Wire Wire Line
 	5300 3500 5300 2600
@@
 Connection ~ 5750 2700
 Wire Wire Line
-	5750 2700 4550 2700
+	5750 2700 5550 2700
 Wire Wire Line
 	6100 3500 6100 2700
-Wire Wire Line
-	5750 2700 6100 2700
 Connection ~ 6100 2700
 Wire Wire Line
@@
 	6500 3300 7350 3300
 Wire Wire Line
-	3500 4450 3500 3200
+	3500 4450 3500 4150
 Connection ~ 3500 3200
 NoConn ~ 6550 4100
@@
 Text Label 2800 3600 0    50   ~ 0
 IB5
+$Comp
+L Device:R R5
+U 1 1 64841BF2
+P 4200 3650
+F 0 "R5" V 3993 3650 50  0000 C CNN
+F 1 "56k" V 4084 3650 50  0000 C CNN
+F 2 "Resistor_THT:R_Axial_DIN0207_L6.3mm_D2.5mm_P7.62mm_Horizontal" V 4130 3650 50  0001 C CNN
+F 3 "~" H 4200 3650 50  0001 C CNN
+	1    4200 3650
+	0    1    1    0
+$EndComp
+$Comp
+L Device:R R6
+U 1 1 64843BDC
+P 4200 4150
+F 0 "R6" V 3993 4150 50  0000 C CNN
+F 1 "56k" V 4084 4150 50  0000 C CNN
+F 2 "Resistor_THT:R_Axial_DIN0207_L6.3mm_D2.5mm_P7.62mm_Horizontal" V 4130 4150 50  0001 C CNN
+F 3 "~" H 4200 4150 50  0001 C CNN
+	1    4200 4150
+	0    1    1    0
+$EndComp
+$Comp
+L Device:R R7
+U 1 1 648441E6
+P 5550 4200
+F 0 "R7" H 5620 4246 50  0000 L CNN
+F 1 "560" H 5620 4155 50  0000 L CNN
+F 2 "Resistor_THT:R_Axial_DIN0207_L6.3mm_D2.5mm_P7.62mm_Horizontal" V 5480 4200 50  0001 C CNN
+F 3 "~" H 5550 4200 50  0001 C CNN
+	1    5550 4200
+	1    0    0    -1
+$EndComp
+$Comp
+L Device:R R8
+U 1 1 6484513E
+P 5950 3050
+F 0 "R8" H 6020 3096 50  0000 L CNN
+F 1 "560" H 6020 3005 50  0000 L CNN
+F 2 "Resistor_THT:R_Axial_DIN0207_L6.3mm_D2.5mm_P7.62mm_Horizontal" V 5880 3050 50  0001 C CNN
+F 3 "~" H 5950 3050 50  0001 C CNN
+	1    5950 3050
+	1    0    0    -1
+$EndComp
+Wire Wire Line
+	5750 2700 5950 2700
+Connection ~ 5950 2700
+Wire Wire Line
+	5950 2700 6100 2700
+Wire Wire Line
+	5950 2900 5950 2700
+Wire Wire Line
+	5950 3200 5950 4000
+Connection ~ 5950 4000
+Wire Wire Line
+	5950 4000 6100 4000
+Wire Wire Line
+	5550 4050 5550 2700
+Connection ~ 5550 2700
+Wire Wire Line
+	5550 2700 4550 2700
+Wire Wire Line
+	5550 4350 5550 4450
+Connection ~ 5550 4450
+Wire Wire Line
+	5550 4450 5750 4450
+Wire Wire Line
+	4050 3650 3600 3650
+Connection ~ 3600 3650
+Wire Wire Line
+	3600 3650 3600 4000
+Wire Wire Line
+	4350 3650 4450 3650
+Wire Wire Line
+	4450 3650 4450 4000
+Connection ~ 4450 4000
+Wire Wire Line
+	4050 4150 3500 4150
+Connection ~ 3500 4150
+Wire Wire Line
+	3500 4150 3500 3200
+Wire Wire Line
+	4350 4150 4450 4150
+Wire Wire Line
+	4450 4150 4450 4450
+Connection ~ 4450 4450
 $EndSCHEMATC
